Commit message: Drive robot and create world for gazebo

File: description/robot.urdf.xacro (robot description, xacro)
@@ -2,3 +2,4 @@
 <robot xmlns:xacro="http://www.ros.org/wiki/xacro"  name="robot">
     <xacro:include filename="robot_core.xacro" />
+    <xacro:include filename="gazebo_control.xacro"/>
 </robot>

File: description/robot_core.xacro (robot description, xacro)
@@ -27,14 +27,26 @@
             <origin xyz="0 0 0"/>
             <geometry>
-                <box size="0.12 0.12 0.1"/>
+                <box size="0.12 0.12 0.08"/>
             </geometry>
-            <material name="blue"/>
+            <material name="black"/>
         </visual>
+         <collision>
+            <origin xyz=" 0 0 0"/>
+            <geometry>
+                <box size="0.12 0.12 0.08"/>
+            </geometry>
+        </collision>
+        <xacro:inertial_box mass="0.5" x="0.12" y="0.12" z="0.08">
+            <origin xyz="0 0 0" rpy="0 0 0"/>
+        </xacro:inertial_box>
     </link>
+    <gazebo reference="chassis">
+        <material>Gazebo/White</material>
+    </gazebo>
     <!-- LEFT FRONT WHEEL LINK -->
     <joint name="left_wheel_front_joint" type="continuous">
         <parent link="base_link"/>
         <child link="left_front_wheel"/>
-        <origin xyz="-0.03 -0.073 -0.05" rpy="-${pi/2} 0 0" />
+        <origin xyz="0.03 -0.073 -0.03" rpy="-${pi/2} 0 0" />
         <axis xyz="0 0 1"/>
     </joint>
@@ -55,9 +67,12 @@
         </xacro:inertial_cylinder>
     </link>
+    <gazebo reference="left_front_wheel">
+        <material>Gazebo/Orange</material>
+    </gazebo>
     <!-- LEFT REAR WHEEL LINK -->
     <joint name="left_wheel_rear_joint" type="continuous">
         <parent link="base_link"/>
         <child link="left_rear_wheel"/>
-        <origin xyz="0.05 -0.073 -0.05" rpy="-${pi/2} 0 0" />
+        <origin xyz="-0.05 -0.073 -0.03" rpy="-${pi/2} 0 0" />
         <axis xyz="0 0 1"/>
     </joint>
@@ -78,9 +93,12 @@
         </xacro:inertial_cylinder>
     </link>
+    <gazebo reference="left_rear_wheel">
+        <material>Gazebo/Orange</material>
+    </gazebo>
         <!-- RIGHT FRONT WHEEL LINK -->
     <joint name="right_wheel_front_joint" type="continuous">
         <parent link="base_link"/>
         <child link="right_front_wheel"/>
-        <origin xyz="-0.03 0.073 -0.05" rpy="${pi/2} 0 0" />
+        <origin xyz="0.03 0.073 -0.03" rpy="${pi/2} 0 0" />
         <axis xyz="0 0 -1"/>
     </joint>
@@ -101,10 +119,14 @@
         </xacro:inertial_cylinder>
     </link>
+    <gazebo reference="right_front_wheel">
+        <material>Gazebo/Orange</material>
+    </gazebo>
         <!-- RIGHT REAR WHEEL LINK -->
     <joint name="right_wheel_rear_joint" type="continuous">
         <parent link="base_link"/>
         <child link="right_rear_wheel"/>
-        <origin xyz="0.05 0.073 -0.05" rpy="${pi/2} 0 0" />
+        <origin xyz="-0.05 0.073 -0.03" rpy="${pi/2} 0 0" />
         <axis xyz="0 0 -1"/>
+        <joint_properties damping="1.0" friction="1.0"/>
     </joint>
     <link name="right_rear_wheel">
@@ -124,3 +146,6 @@
         </xacro:inertial_cylinder>
     </link>
+    <gazebo reference="right_rear_wheel">
+        <material>Gazebo/Orange</material>
+    </gazebo>
 </robot>
